File: example/example/example.kicad_pcb (KiCad board)
At the start: 2 copper layers, 98 parts, among them K1 KEYSW, K10 KEYSW, K11 KEYSW, K12 KEYSW, K13 KEYSW, K14 KEYSW, K15 KEYSW, K16 KEYSW, K17 KEYSW, K18 KEYSW, K19 KEYSW, K2 KEYSW, K20 KEYSW, K21 KEYSW, K22 KEYSW, K23 KEYSW, K24 KEYSW, K25 KEYSW, K26 KEYSW, K27 KEYSW, K28 KEYSW, K29 KEYSW, K3 KEYSW, K30 KEYSW, K31 KEYSW, K32 KEYSW, K33 KEYSW, K34 KEYSW, K35 KEYSW, K36 KEYSW, K37 KEYSW, K38 KEYSW, K39 KEYSW, K4 KEYSW, K40 KEYSW, K41 KEYSW, K42 KEYSW, K43 KEYSW, K44 KEYSW, K45 KEYSW, K46 KEYSW, K47 KEYSW, K48 KEYSW, K5 KEYSW, K6 KEYSW, K7 KEYSW, K8 KEYSW, K9 KEYSW, SW1 SW_Push, U1 ProMicro

Commit message: Kicad template 4x12 not wired
Parts:
- D1, D10, D11, D12, D13, D14, D15, D16, D17, D18, D19, D2, D20, D21, D22, D23, D24, D25, D26, D27, D28, D29, D3, D30, D31, D32, D33, D34, D35, D36, D37, D38, D39, D4, D40, D41, D42, D43, D44, D45, D46, D47, D48, D5, D6, D7, D8, D9: moved to B.Cu
- SW1: footprint Button_Switch_THT:SW_PUSH_6mm_H5mm -> Connector_PinHeader_2.54mm:PinHeader_2x01_P2.54mm_Vertical; moved to B.Cu
- moved U1 108.9 mm to (76.2, 47.0)
- moved SW1 57.6 mm to (65.8, 57.1), turned to 90 degrees
- moved D1 27.7 mm to (45.7, 47.8), turned to 180 degrees
- moved D13 25.8 mm to (45.0, 66.8), turned to 180 degrees
- moved D25 25.1 mm to (45.5, 85.6), turned to 180 degrees
- moved K12 25.0 mm to (250.2, 33.0)
- moved D37 24.1 mm to (46.2, 100.3)
- moved K24 24.1 mm to (250.2, 52.1)
- moved D12 23.7 mm to (238.3, 43.2)
- moved K36 23.4 mm to (250.2, 71.1)
- moved D24 23.0 mm to (238.0, 62.2)
- moved K48 23.0 mm to (250.2, 90.2)
- moved K11 22.7 mm to (231.1, 33.0)
- moved D36 22.1 mm to (238.3, 81.3)
- moved D48 21.9 mm to (238.0, 100.3)
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Connections:
- K15 pad 2: Net-(K15-Pad2) -> Net-(D15-Pad2)
Routing:
- net row2: track 0.00 -> 195.0 mm
- net row3: track 0.00 -> 191.8 mm
- net row1: track 0.00 -> 169.1 mm
- net row0: track 0.00 -> 147.1 mm
- net col10: track 0.00 -> 100.8 mm
- net col2: track 0.00 -> 78.2 mm, vias 0 -> 2
- net col1: track 0.00 -> 78.0 mm, vias 0 -> 2
- net col11: track 0.00 -> 75.9 mm
- net col0: track 0.00 -> 59.9 mm
- net col3: track 0.00 -> 22.3 mm
- net Net-(D37-Pad2): track 0.00 -> 21.4 mm
- net Net-(D4-Pad2): track 0.00 -> 14.3 mm
- net Net-(D1-Pad2): track 0.00 -> 14.2 mm
- net Net-(D13-Pad2): track 0.00 -> 13.5 mm
- net Net-(D25-Pad2): track 0.00 -> 13.4 mm
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Other:
- board outline added: 231 x 76.2 mm
- net class Default: trace_width 0.25 -> 1.2; via_dia 0.8 -> 1.2; via_drill 0.4 -> 0.6
